File: 3_Hardware/KiCad/GPS-MINPOINT.kicad_sch (KiCad schematic)
At the start: 23 parts, among them J1 110990030, U2 PIC24FJ64GA002-I/SP

Commit message: Upload of finished PCB design
Parts:
- removed D3, D4, D5, D6, D7, D8: LED, symbol Device:LED
- removed D9: G_LED, symbol Device:LED
- removed R4, R5, R6, R7, R8, R9: R, symbol Device:R
- added C4, C5: 10uF, Capacitor_THT:C_Disc_D4.7mm_W2.5mm_P5.00mm, symbol Device:C
- added J2: LCD, Connector_PinSocket_2.54mm:PinSocket_1x05_P2.54mm_Vertical, symbol Connector_Generic:Conn_01x05
- added J3: ProgrammerConnector, Connector_PinHeader_2.54mm:PinHeader_1x08_P2.54mm_Vertical, symbol Connector_Generic:Conn_01x08
- added J4: PWR, Connector_PinHeader_2.54mm:PinHeader_1x01_P2.54mm_Vertical, symbol Connector_Generic:Conn_01x01
- C1: value C -> 10uF; footprint (none) -> Capacitor_THT:C_Disc_D4.7mm_W2.5mm_P5.00mm
- C2, C3: value C -> 100nF; footprint (none) -> Capacitor_THT:C_Disc_D4.7mm_W2.5mm_P5.00mm
- D1: value LED -> G_LED; footprint (none) -> LED_THT:LED_D3.0mm
- D2: value LED -> R_LED; footprint (none) -> LED_THT:LED_D3.0mm
- R1, R2: value R -> 220; footprint (none) -> Resistor_THT:R_Axial_DIN0207_L6.3mm_D2.5mm_P7.62mm_Horizontal
- R3: value R -> 10k; footprint (none) -> Resistor_THT:R_Axial_DIN0207_L6.3mm_D2.5mm_P7.62mm_Horizontal
Connections:
- net at D1.1 (K): now also U2.2
- net at R1.1: now also C1.1, C2.1, C3.1, J1.2 (VCC), R2.1, R3.2, U2.13, U2.28, C5.1, J2.2 (VDD), J3.2 (Pin_2), J4.1 (Pin_1)
- net at R3.1: now also U2.1, J3.1 (Pin_1)
- net at C1.2, C2.2, C3.2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: now also D2.1 (K), J1.1 (GND), U2.19, C4.2, C5.2, J2.3 (GND), J3.3 (Pin_3); no longer J1.4 (GND)
- net at U2.21: now also J1.4 (TX); no longer J1.1 (TX)
- net at U2.15: now also J1.3 (RX); no longer J1.2 (RX)
- net at U2.20: now also C4.1
- net at U2.4: now also J3.4 (Pin_4)
- net at U2.5: now also J3.5 (Pin_5)
- net at U2.6: now also J2.4 (SDA)
- net at U2.7: now also J2.5 (SCL)
Other:
- title: (none) -> GPS-MINPOINT SCHEMATIC
- moved on the sheet: C1, C2, C3, D1, J1, R1, U2
